File: Artix7_SOM/Artix7_SOM.kicad_sch (KiCad schematic)
At the start: 0 parts

Commit message: update
Other:
- added sheet connectors (connector.kicad_sch)
- added sheet mgt (mgt.kicad_sch)
- added sheet pinout2 (pinout2.kicad_sch)
Changed lines of the file:
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@@
 (kicad_sch (version 20230121) (generator eeschema)
   (paper "A4")
-  (sheet (at 74.93 48.26) (size 25.4 15.24) (fields_autoplaced)
+  (sheet (at 96.52 64.77) (size 25.4 15.24) (fields_autoplaced)
     (stroke (width 0.1524) (type solid))
     (fill (color 0 0 0 0.0000))
-    (property "Sheetname" "pinout" (at 74.93 47.5484 0)
+    (property "Sheetname" "pinout" (at 96.52 64.0584 0)
       (effects (font (size 1.27 1.27)) (justify left bottom))
     )
-    (property "Sheetfile" "pinout.kicad_sch" (at 74.93 64.0846 0)
+    (property "Sheetfile" "pinout.kicad_sch" (at 96.52 80.5946 0)
       (effects (font (size 1.27 1.27)) (justify left top))
     )
@@
     )
   )
-  (sheet (at 110.49 48.26) (size 22.86 15.24) (fields_autoplaced)
+  (sheet (at 132.08 64.77) (size 22.86 15.24) (fields_autoplaced)
     (stroke (width 0.1524) (type solid))
     (fill (color 0 0 0 0.0000))
-    (property "Sheetname" "config" (at 110.49 47.5484 0)
+    (property "Sheetname" "config" (at 132.08 64.0584 0)
       (effects (font (size 1.27 1.27)) (justify left bottom))
     )
-    (property "Sheetfile" "config.kicad_sch" (at 110.49 64.0846 0)
+    (property "Sheetfile" "config.kicad_sch" (at 132.08 80.5946 0)
+      (effects (font (size 1.27 1.27)) (justify left top))
+    )
+    (instances
+      (project "Artix7_SOM"
+        (path "/de078e16-8db1-4ffc-8e44-4cf56292f9f1" (page "5"))
+      )
+    )
+  )
+  (sheet (at 63.5 90.17) (size 25.4 16.51) (fields_autoplaced)
+    (stroke (width 0.1524) (type solid))
+    (fill (color 0 0 0 0.0000))
+    (property "Sheetname" "mgt" (at 63.5 89.4584 0)
+      (effects (font (size 1.27 1.27)) (justify left bottom))
+    )
+    (property "Sheetfile" "mgt.kicad_sch" (at 63.5 107.2646 0)
+      (effects (font (size 1.27 1.27)) (justify left top))
+    )
+    (instances
+      (project "Artix7_SOM"
+        (path "/de078e16-8db1-4ffc-8e44-4cf56292f9f1" (page "6"))
+      )
+    )
+  )
+  (sheet (at 134.62 92.71) (size 24.13 15.24) (fields_autoplaced)
+    (stroke (width 0.1524) (type solid))
+    (fill (color 0 0 0 0.0000))
+    (property "Sheetname" "connectors" (at 134.62 91.9984 0)
+      (effects (font (size 1.27 1.27)) (justify left bottom))
+    )
+    (property "Sheetfile" "connector.kicad_sch" (at 134.62 108.5346 0)
+      (effects (font (size 1.27 1.27)) (justify left top))
+    )
+    (instances
+      (project "Artix7_SOM"
+        (path "/de078e16-8db1-4ffc-8e44-4cf56292f9f1" (page "7"))
+      )
+    )
+  )
+  (sheet (at 62.23 64.77) (size 22.86 13.97) (fields_autoplaced)
+    (stroke (width 0.1524) (type solid))
+    (fill (color 0 0 0 0.0000))
+    (property "Sheetname" "power" (at 62.23 64.0584 0)
+      (effects (font (size 1.27 1.27)) (justify left bottom))
+    )
+    (property "Sheetfile" "power.kicad_sch" (at 62.23 79.3246 0)
+      (effects (font (size 1.27 1.27)) (justify left top))
+    )
+    (instances
+      (project "Artix7_SOM"
+        (path "/de078e16-8db1-4ffc-8e44-4cf56292f9f1" (page "2"))
+      )
+    )
+  )
+  (sheet (at 96.52 92.71) (size 25.4 15.24) (fields_autoplaced)
+    (stroke (width 0.1524) (type solid))
+    (fill (color 0 0 0 0.0000))
+    (property "Sheetname" "pinout2" (at 96.52 91.9984 0)
+      (effects (font (size 1.27 1.27)) (justify left bottom))
+    )
+    (property "Sheetfile" "pinout2.kicad_sch" (at 96.52 108.5346 0)
       (effects (font (size 1.27 1.27)) (justify left top))
     )
@@
       )
     )
-  )
-  (sheet (at 40.64 48.26) (size 22.86 13.97) (fields_autoplaced)
-    (stroke (width 0.1524) (type solid))
-    (fill (color 0 0 0 0.0000))
-    (property "Sheetname" "power" (at 40.64 47.5484 0)
-      (effects (font (size 1.27 1.27)) (justify left bottom))
-    )
-    (property "Sheetfile" "power.kicad_sch" (at 40.64 62.8146 0)
-      (effects (font (size 1.27 1.27)) (justify left top))
-    )
-    (instances
-      (project "Artix7_SOM"
-        (path "/de078e16-8db1-4ffc-8e44-4cf56292f9f1" (page "2"))
-      )
-    )
