File: Artix7_SOM/config.kicad_sch (KiCad schematic)
At the start: 0 parts

Commit message: update
Parts:
- added U1: XC7A100T-FGG676, Package_BGA:Xilinx_FGG676, symbol FPGA_Xilinx_Artix7:XC7A100T-FGG676
Connections:
- new net TDO: U1.J10 (TDO_0)
