File: Artix7_SOM/pinout.kicad_sch (KiCad schematic)
At the start: 0 parts

Commit message: update
Parts:
- added U1: XC7A100T-FGG676, Package_BGA:Xilinx_FGG676, symbol FPGA_Xilinx_Artix7:XC7A100T-FGG676
Connections:
- new net +3V3: U1.AA21 (VCCO_12), U1.AB18 (VCCO_12), U1.AC25 (VCCO_13), U1.AD22 (VCCO_12), U1.AE19 (VCCO_12), U1.AF26 (VCCO_12), U1.F26 (VCCO_15), U1.G23 (VCCO_15), U1.H20 (VCCO_15), U1.J17 (VCCO_15), U1.K14 (VCCO_15), U1.K24 (VCCO_14), U1.L21 (VCCO_14), U1.M18 (VCCO_15), U1.N15 (VCCO_14), U1.N25 (VCCO_14), U1.P22 (VCCO_14), U1.R19 (VCCO_14), U1.T16 (VCCO_13), U1.T26 (VCCO_13), U1.U23 (VCCO_13), U1.V20 (VCCO_13), U1.W17 (VCCO_12), U1.Y24 (VCCO_13)
