File: Artix7_SOM/pinout2.kicad_sch (KiCad schematic)
At the start: 1 part, among them U1 XC7A100T-FGG676

Commit message: update
Parts:
- removed U1: XC7A100T-FGG676, Package_BGA:Xilinx_FGG676, symbol FPGA_Xilinx_Artix7:XC7A100T-FGG676
- added U1: XC7A100T-FGG676, Package_BGA:Xilinx_FGG676, symbol FPGA_Xilinx_Artix7:XC7A100T-FGG676
Connections:
- new net +3V3: U1.A1 (VCCO_35), U1.A21 (VCCO_16), U1.AA1 (VCCO_33), U1.AC5 (VCCO_33), U1.AD2 (VCCO_33), U1.B18 (VCCO_16), U1.C25 (VCCO_16), U1.C5 (VCCO_35), U1.D2 (VCCO_35), U1.D22 (VCCO_16), U1.E19 (VCCO_16), U1.F16 (VCCO_16), U1.F6 (VCCO_35), U1.G3 (VCCO_35), U1.J7 (VCCO_35), U1.K4 (VCCO_34), U1.L1 (VCCO_34), U1.M8 (VCCO_34), U1.N5 (VCCO_34), U1.P2 (VCCO_34), U1.T6 (VCCO_34), U1.U3 (VCCO_33), U1.W7 (VCCO_33), U1.Y4 (VCCO_33)
