File: Artix_SOM/Artix_SOM/pinout.kicad_sch (KiCad schematic)
At the start: 1 part, among them U1 XC7A100T-FGG676

Commit message: update
Changed lines of the file:
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@@
 	(wire
 		(pts
-			(xy 232.41 119.38) (xy 241.3 119.38)
+			(xy 231.14 119.38) (xy 241.3 119.38)
 		)
 		(stroke
@@
 	(global_label "FPGA_CSO"
 		(shape bidirectional)
-		(at 232.41 119.38 180)
-		(effects
-			(font
-				(size 1.27 1.27)
-			)
-			(justify right)
-		)
-		(property "Intersheetrefs" "${INTERSHEET_REFS}"
-			(at 232.41 119.38 0)
-			(effects
-				(font
+		(at 231.14 119.38 180)
+		(effects
+			(font
+				(size 1.27 1.27)
+			)
+			(justify right)
+		)
+		(property "Intersheetrefs" "${INTERSHEET_REFS}"
+			(at 231.14 119.38 0)
+			(effects
+				(font

Commit message: update
Connections:
- no-connect marks 0 -> 6
Changed lines of the file:
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@@
 		(color 0 0 0 0)
+	)
+	(no_connect
+		(at 342.9 215.9)
+	)
+	(no_connect
+		(at 342.9 91.44)
+	)
+	(no_connect
+		(at 241.3 91.44)
+	)
+	(no_connect
+		(at 163.83 90.17)
+	)
+	(no_connect
+		(at 241.3 215.9)
+	)
+	(no_connect
+		(at 163.83 214.63)
 	)
 	(wire
