File: Artix_SOM/Artix_SOM/config.kicad_sch (KiCad schematic)
At the start: 14 parts, among them SW1 SW_Push, U1 XC7A100T-FGG676

Commit message: update
Parts:
- R2: value R_US -> 4,7k
Changed lines of the file:
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@@
 			)
 		)
-		(property "Value" "R_US"
+		(property "Value" "4,7k"
 			(at 189.23 102.8699 0)
 			(effects
