File: Artix_SOM/Artix_SOM/pinout2.kicad_sch (KiCad schematic)
At the start: 1 part, among them U1 XC7A100T-FGG676

Commit message: update
Parts:
- added R6: R_US, symbol Device:R_US
- added SW2: SW_Push, symbol Switch:SW_Push
Connections:
- net +3V3: now also R6.1
- net at U1.J8 (IO_0_35): now also R6.2, SW2.2
- new net GND: SW2.1

Commit message: update
Connections:
- net ~{RESET}: now reaches U1.H17 (IO_0_16)
- net B16_L10_N renamed DQ12
- net B16_L10_P renamed DQ11
- net B16_L11_N renamed DQ14
- net B16_L11_P renamed DQ13
- net B16_L12_N renamed UDQS
- net B16_L12_P renamed DQ15
- net B16_L13_N renamed LDQS
- net B16_L13_P renamed ~{UDQS}
- net B16_L14_N renamed UDM
- net B16_L14_P renamed ~{LDQS}
- net B16_L15_N renamed A0
- net B16_L15_P renamed LDM
- net B16_L16_N renamed A2
- net B16_L16_P renamed A1
- net B16_L17_N renamed A4
- net B16_L17_P renamed A3
- net B16_L18_N renamed A6
- net B16_L18_P renamed A5
- net B16_L19_N renamed A8
- net B16_L19_P renamed A7
- net B16_L1_N renamed ~{CK}
- net B16_L1_P renamed CK
- net B16_L20_N renamed A10/AP
- net B16_L20_P renamed A9
- net B16_L21_N renamed A12/~{BC}
- net B16_L21_P renamed A11
- net B16_L22_N renamed BA0
- net B16_L22_P renamed A13
- net B16_L23_N renamed BA2
- net B16_L23_P renamed BA1
- net B16_L24_N: no longer names the net of U1.D24 (IO_L24N_T3_16)
- net B16_L24_P renamed ODT
- net B16_L2_N renamed ~{CS}
- net B16_L2_P renamed CKE
- net B16_L3_N renamed ~{CAS}
- net B16_L3_P renamed ~{RAS}
- net B16_L4_N renamed DQ0
- net B16_L4_P renamed ~{WE}
- net B16_L5_N renamed DQ2
- net B16_L5_P renamed DQ1
- net B16_L6_N renamed DQ4
- net B16_L6_P renamed DQ3
- net B16_L7_N renamed DQ6
- net B16_L7_P renamed DQ5
- net B16_L8_N renamed DQ8
- net B16_L8_P renamed DQ7
- net B16_L9_N renamed DQ10
- net B16_L9_P renamed DQ9
- no-connect marks 0 -> 5

Commit message: update
Other:
- note added: "CLK 100MHz"
- note added: "DDR pins"
- note added: "RESETN"
Changed lines of the file:
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@@
+		)
+	)
+	(rectangle
+		(start 368.3 148.59)
+		(end 392.43 156.21)
+		(stroke
+			(width 0)
+			(type dash)
+		)
+		(fill
+			(type none)
+		)
+	)
+	(rectangle
+		(start 45.72 80.01)
+		(end 72.39 218.44)
+		(stroke
+			(width 0)
+			(type dash)
+		)
+		(fill
+			(type none)
+		)
+	)
+	(rectangle
+		(start 364.49 73.66)
+		(end 382.27 119.38)
+		(stroke
+			(width 0)
+			(type dash)
+		)
+		(fill
+			(type none)
+		)
+	)
+	(text "RESETN"
+		(exclude_from_sim no)
+		(at 367.792 72.644 0)
+		(effects
+			(font
+				(size 1.27 1.27)
+			)
+		)
+	)
+	(text "CLK 100MHz"
+		(exclude_from_sim no)
+		(at 374.396 147.32 0)
+		(effects
+			(font
+				(size 1.27 1.27)
+			)
+		)
+	)
+	(text "DDR pins"
+		(exclude_from_sim no)
+		(at 56.388 82.55 0)
+		(effects
+			(font
+				(size 1.27 1.27)
+			)
 		)
 	)
