File: Artix_SOM/Artix_SOM/connectors.kicad_sch (KiCad schematic)
At the start: 2 parts

Commit message: update
Connections:
- net +5V: now reaches J1.1
- net +5V: now also J1.2, J1.3, J1.4, J1.5, J1.6
- net B14_L15_P: now reaches J1.10
- net B14_L4_N: now reaches J1.11
- net TMS: now reaches J1.111
- net TDI: now reaches J1.112
- net TCK: now reaches J1.113
- net TDO: now reaches J1.114
- net GND: now reaches J1.115
- net GND: now also J1.116, J1.117, J1.118, J1.119, J1.40
- net B14_L15_N: now reaches J1.12
- net B14_L5_P: now reaches J1.13
- net B14_L16_P: now reaches J1.14
- net B14_L5_N: now reaches J1.15
- net B14_L16_N: now reaches J1.16
- net B14_L6_N: now reaches J1.17
- net B14_L17_P: now reaches J1.18
- net B14_L7_P: now reaches J1.19
- net B14_L17_N: now reaches J1.20
- net B14_L7_N: now reaches J1.21
- net B14_L18_P: now reaches J1.22
- net B14_L8_P: now reaches J1.23
- net B14_L18_N: now reaches J1.24
- net B14_L8_N: now reaches J1.25
- net B14_L19_P: now reaches J1.26
- net B14_L9_P: now reaches J1.27
- net B14_L19_N: now reaches J1.28
- net B14_L9_N: now reaches J1.29
- net B14_L20_P: now reaches J1.30
- net B14_L10_P: now reaches J1.31
- net B14_L20_N: now reaches J1.32
- net B14_L10_N: now reaches J1.33
- net B14_L21_P: now reaches J1.34
- net B14_L11_P: now reaches J1.35
- net B14_L21_N: now reaches J1.36
- net B14_L11_N: now reaches J1.37
- net B14_L22_P: now reaches J1.38
- net B14_L12_P: now reaches J1.39
- net B14_L12_N: now reaches J1.41
- net B14_L23_P: now reaches J1.42
- net B14_L13_P: now reaches J1.43
- net B14_L23_N: now reaches J1.44
- net B14_L13_N: now reaches J1.45
- net B14_L24_P: now reaches J1.46
- net B14_L14_P: now reaches J1.47
- net B14_L24_N: now reaches J1.48
- net B14_L3_N: now reaches J1.7
- net B14_L14_N: now reaches J1.8
- net B14_L4_P: now reaches J1.9
- net B15_L1_P: now reaches J2.1
- net B34_L3_P: now reaches J2.10
- net B15_L3_N: now reaches J2.11
- net VN: now reaches J2.119
- net B34_L3_N: now reaches J2.12
- net B15_L4_P: now reaches J2.13
- net B34_L4_P: now reaches J2.14
- net B15_L4_N: now reaches J2.15
- net B34_L4_N: now reaches J2.16
- net B15_L5_P: now reaches J2.17
- net B34_L5_P: now reaches J2.18
- net B15_L5_N: now reaches J2.19
- net B34_L1_P: now reaches J2.2
- net B34_L5_N: now reaches J2.20
- net B15_L6_P: now reaches J2.21
- net B34_L6_P: now reaches J2.22
- net B15_L6_N: now reaches J2.23
- net B34_L6_N: now reaches J2.24
- net B15_L7_P: now reaches J2.25
- net B34_L7_P: now reaches J2.26
- net B15_L7_N: now reaches J2.27
- net B34_L7_N: now reaches J2.28
- net B15_L8_P: now reaches J2.29
- net B15_L1_N: now reaches J2.3
- net B34_L8_P: now reaches J2.30
- net B15_L8_N: now reaches J2.31
- net B34_L8_N: now reaches J2.32
- net B15_L9_P: now reaches J2.33
- net B34_L9_P: now reaches J2.34
- net B15_L9_N: now reaches J2.35
- net B34_L9_N: now reaches J2.36
- net B15_L10_P: now reaches J2.37
- net B34_L10_P: now reaches J2.38
- net B15_L10_N: now reaches J2.39
- net B34_L1_N: now reaches J2.4
- net VP: now reaches J2.40
- net B15_L11_P: now reaches J2.41
- net B34_L11_P: now reaches J2.42
- net B15_L11_N: now reaches J2.43
- net B34_L11_N: now reaches J2.44
- net B15_L12_P: now reaches J2.45
- net B34_L12_P: now reaches J2.46
- net B15_L12_N: now reaches J2.47
- net B34_L12_N: now reaches J2.48
- net B15_L13_P: now reaches J2.49
- net B15_L2_P: now reaches J2.5
- net B34_L13_P: now reaches J2.50
- net B15_L13_N: now reaches J2.51
- net B34_L13_N: now reaches J2.52
- net B15_L14_P: now reaches J2.53
- net B34_L14_P: now reaches J2.54
- net B15_L14_N: now reaches J2.55
- net B34_L14_N: now reaches J2.56
- net B15_L15_P: now reaches J2.57
- net B34_L15_P: now reaches J2.58
- net B15_L15_N: now reaches J2.59
- net B34_L2_P: now reaches J2.6
- net B34_L15_N: now reaches J2.60
- net B15_L16_P: now reaches J2.61
- net B34_L16_P: now reaches J2.62
- net B15_L16_N: now reaches J2.63
- net B34_L16_N: now reaches J2.64
- net B15_L17_P: now reaches J2.65
- net B34_L17_P: now reaches J2.66
- net B15_L17_N: now reaches J2.67
- net B34_L17_N: now reaches J2.68
- net B15_L18_P: now reaches J2.69
- net B15_L2_N: now reaches J2.7
- net B34_L18_P: now reaches J2.70
- net B15_L18_N: now reaches J2.71
- net B34_L18_N: now reaches J2.72
- net B15_L19_P: now reaches J2.73
- net B34_L19_P: now reaches J2.74
- net B15_L19_N: now reaches J2.75
- net B34_L19_N: now reaches J2.76
- net B15_L20_P: now reaches J2.77
- net B34_L20_P: now reaches J2.78
- net B15_L20_N: now reaches J2.79
- net B34_L2_N: now reaches J2.8
- net B34_L20_N: now reaches J2.80
- net B15_L21_P: now reaches J2.81
- net B34_L21_P: now reaches J2.82
- net B15_L21_N: now reaches J2.83
- net B34_L21_N: now reaches J2.84
- net B15_L22_P: now reaches J2.85
- net B34_L22_P: now reaches J2.86
- net B15_L22_N: now reaches J2.87
- net B34_L22_N: now reaches J2.88
- net B15_L23_P: now reaches J2.89
- net B15_L3_P: now reaches J2.9
- net B34_L23_P: now reaches J2.90
- net B15_L23_N: now reaches J2.91
- net B34_L23_N: now reaches J2.92
- net B15_L24_P: now reaches J2.93
- net B34_L24_P: now reaches J2.94
- net B15_L24_N: now reaches J2.95
- net B34_L24_N: now reaches J2.96
- new net B14_L22_N: J1.40
- new net B34_L10_N: J2.40
- no-connect marks 0 -> 84

Commit message: update
Parts:
- removed J2: ~, symbol Panasonic_connector:AXK6A2337YG
- added unit 2 of J1
- J1: symbol Panasonic_connector:AXK6A2337YG -> SOM_library:SoM_male
Connections:
- net B15_L10_N: now also J1.39 (PIN39_B2)
- net B15_L10_P: now also J1.37 (PIN37_B2)
- net B15_L11_N: now also J1.43 (PIN43_B2)
- net B15_L11_P: now also J1.41 (PIN41_B2)
- net B15_L12_N: now also J1.47 (PIN47_B2)
- net B15_L12_P: now also J1.45 (PIN45_B2)
- net B15_L13_N: now also J1.51 (PIN51_B2)
- net B15_L13_P: now also J1.49 (PIN49_B2)
- net B15_L14_N: now also J1.55 (PIN55_B2)
- net B15_L14_P: now also J1.53 (PIN53_B2)
- net B15_L15_N: now also J1.59 (PIN59_B2)
- net B15_L15_P: now also J1.57 (PIN57_B2)
- net B15_L16_N: now also J1.63 (PIN63_B2)
- net B15_L16_P: now also J1.61 (PIN61_B2)
- net B15_L17_N: now also J1.67 (PIN67_B2)
- net B15_L17_P: now also J1.65 (PIN65_B2)
- net B15_L18_N: now also J1.71 (PIN71_B2)
- net B15_L18_P: now also J1.69 (PIN69_B2)
- net B15_L19_N: now also J1.75 (PIN75_B2)
- net B15_L19_P: now also J1.73 (PIN73_B2)
- net B15_L1_N: now also J1.3 (PIN3_B2)
- net B15_L1_P: now also J1.1 (PIN1_B2)
- net B15_L20_N: now also J1.79 (PIN79_B2)
- net B15_L20_P: now also J1.77 (PIN77_B2)
- net B15_L21_N: now also J1.83 (PIN83_B2)
- net B15_L21_P: now also J1.81 (PIN81_B2)
- net B15_L22_N: now also J1.87 (PIN87_B2)
- net B15_L22_P: now also J1.85 (PIN85_B2)
- net B15_L23_N: now also J1.91 (PIN91_B2)
- net B15_L23_P: now also J1.89 (PIN89_B2)
- net B15_L24_N: now also J1.95 (PIN95_B2)
- net B15_L24_P: now also J1.93 (PIN93_B2)
- net B15_L2_N: now also J1.7 (PIN7_B2)
- net B15_L2_P: now also J1.5 (PIN5_B2)
- net B15_L3_N: now also J1.11 (PIN11_B2)
- net B15_L3_P: now also J1.9 (PIN9_B2)
- net B15_L4_N: now also J1.15 (PIN15_B2)
- net B15_L4_P: now also J1.13 (PIN13_B2)
- net B15_L5_N: now also J1.19 (PIN19_B2)
- net B15_L5_P: now also J1.17 (PIN17_B2)
- net B15_L6_N: now also J1.23 (PIN23_B2)
- net B15_L6_P: now also J1.21 (PIN21_B2)
- net B15_L7_N: now also J1.27 (PIN27_B2)
- net B15_L7_P: now also J1.25 (PIN25_B2)
- net B15_L8_N: now also J1.31 (PIN31_B2)
- net B15_L8_P: now also J1.29 (PIN29_B2)
- net B15_L9_N: now also J1.35 (PIN35_B2)
- net B15_L9_P: now also J1.33 (PIN33_B2)
- net B34_L10_N: now also J1.40 (PIN40_B2)
- net B34_L10_P: now also J1.38 (PIN38_B2)
- net B34_L11_N: now also J1.44 (PIN44_B2)
- net B34_L11_P: now also J1.42 (PIN42_B2)
- net B34_L12_N: now also J1.48 (PIN48_B2)
- net B34_L12_P: now also J1.46 (PIN46_B2)
- net B34_L13_N: now also J1.52 (PIN52_B2)
- net B34_L13_P: now also J1.50 (PIN50_B2)
- net B34_L14_N: now also J1.56 (PIN56_B2)
- net B34_L14_P: now also J1.54 (PIN54_B2)
- net B34_L15_N: now also J1.60 (PIN60_B2)
- net B34_L15_P: now also J1.58 (PIN58_B2)
- net B34_L16_N: now also J1.64 (PIN64_B2)
- net B34_L16_P: now also J1.62 (PIN62_B2)
- net B34_L17_N: now also J1.68 (PIN68_B2)
- net B34_L17_P: now also J1.66 (PIN66_B2)
- net B34_L18_N: now also J1.72 (PIN72_B2)
- net B34_L18_P: now also J1.70 (PIN70_B2)
- net B34_L19_N: now also J1.76 (PIN76_B2)
- net B34_L19_P: now also J1.74 (PIN74_B2)
- net B34_L1_N: now also J1.4 (PIN4_B2)
- net B34_L1_P: now also J1.2 (PIN2_B2)
- net B34_L20_N: now also J1.80 (PIN80_B2)
- net B34_L20_P: now also J1.78 (PIN78_B2)
- net B34_L21_N: now also J1.84 (PIN84_B2)
- net B34_L21_P: now also J1.82 (PIN82_B2)
- net B34_L22_N: now also J1.88 (PIN88_B2)
- net B34_L22_P: now also J1.86 (PIN86_B2)
- net B34_L23_N: now also J1.92 (PIN92_B2)
- net B34_L23_P: now also J1.90 (PIN90_B2)
- net B34_L24_N: now also J1.96 (PIN96_B2)
- net B34_L24_P: now also J1.94 (PIN94_B2)
- net B34_L2_N: now also J1.8 (PIN8_B2)
- net B34_L2_P: now also J1.6 (PIN6_B2)
- net B34_L3_N: now also J1.12 (PIN12_B2)
- net B34_L3_P: now also J1.10 (PIN10_B2)
- net B34_L4_N: now also J1.16 (PIN16_B2)
- net B34_L4_P: now also J1.14 (PIN14_B2)
- net B34_L5_N: now also J1.20 (PIN20_B2)
- net B34_L5_P: now also J1.18 (PIN18_B2)
- net B34_L6_N: now also J1.24 (PIN24_B2)
- net B34_L6_P: now also J1.22 (PIN22_B2)
- net B34_L7_N: now also J1.28 (PIN28_B2)
- net B34_L7_P: now also J1.26 (PIN26_B2)
- net B34_L8_N: now also J1.32 (PIN32_B2)
- net B34_L8_P: now also J1.30 (PIN30_B2)
- net B34_L9_N: now also J1.36 (PIN36_B2)
- net B34_L9_P: now also J1.34 (PIN34_B2)
- net GND: now also J1.120 (GND); no longer J1.40
- net VN: now also J1.119 (ADC_N)
- net VP: now also J1.120 (ADC_P)
Other:
- moved on the sheet: J1A

Commit message: update
Parts:
- renumbered J1 to J?
Changed lines of the file:
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@@
 		(dnp no)
 		(fields_autoplaced yes)
-		(property "Reference" "J1"
+		(property "Reference" "J?"
 			(at 129.54 53.34 0)
 			(effects
@@
 		(pin "117"
 		)
+		(instances
+			(project "Artix_SOM"
+				(path "/c2221598-f078-4310-82f6-aed2a006194d/12c2dede-18ee-4a62-9b3f-2a242fe2e990"
+					(reference "J?")
+					(unit 1)
+				)
+			)
+		)
 	)

Commit message: update dc source
Connections:
- net +5V renamed +12V
Changed lines of the file:
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@@
 	)
 	(symbol
-		(lib_id "power:+5V")
+		(lib_id "power:+12V")
 		(at 129.54 45.72 0)
 		(unit 1)
@@
 		(dnp no)
 		(fields_autoplaced yes)
-		(property "Reference" "#PWR035"
+		(property "Reference" "#PWR037"
 			(at 129.54 49.53 0)
 			(effects
@@
 			)
 		)
-		(property "Value" "+5V"
+		(property "Value" "+12V"
 			(at 129.54 40.64 0)
 			(effects
@@
 			)
 		)
-		(property "Description" "Power symbol creates a global label with name \"+5V\""
+		(property "Description" "Power symbol creates a global label with name \"+12V\""
 			(at 129.54 45.72 0)
 			(effects
@@
 		)
 		(instances
-			(project "Artix_SOM"
+			(project ""
 				(path "/c2221598-f078-4310-82f6-aed2a006194d/12c2dede-18ee-4a62-9b3f-2a242fe2e990"
-					(reference "#PWR035")
+					(reference "#PWR037")
 					(unit 1)
 				)
