File: Artix_SOM/Artix_SOM/Artix_SOM.kicad_sch (KiCad schematic)
At the start: 0 parts

Commit message: update
Other:
- added sheet ddr (ddr.kicad_sch)
Changed lines of the file:
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@@
+	)
+	(sheet
+		(at 167.64 62.23)
+		(size 29.21 17.78)
+		(fields_autoplaced yes)
+		(stroke
+			(width 0.1524)
+			(type solid)
+		)
+		(fill
+			(color 0 0 0 0.0000)
+		)
+		(property "Sheetname" "ddr"
+			(at 167.64 61.5184 0)
+			(effects
+				(font
+					(size 1.27 1.27)
+				)
+				(justify left bottom)
+			)
+		)
+		(property "Sheetfile" "ddr.kicad_sch"
+			(at 167.64 80.5946 0)
+			(effects
+				(font
+					(size 1.27 1.27)
+				)
+				(justify left top)
+			)
+		)
+		(instances
+			(project "Artix_SOM"
+				(path "/c2221598-f078-4310-82f6-aed2a006194d"
+					(page "9")
+				)
+			)
+		)
 	)
 	(sheet

Commit message: update
Other:
- sheet pinout renamed FPGA_1
- sheet pinout2 renamed FPGA_2
- sheet FPGA_1: file pinout.kicad_sch -> FPGA_1.kicad_sch
- sheet FPGA_2: file pinout2.kicad_sch -> FPGA_2.kicad_sch
Changed lines of the file:
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@@
 			(color 0 0 0 0.0000)
 		)
-		(property "Sheetname" "pinout2"
+		(property "Sheetname" "FPGA_2"
 			(at 100.33 88.1884 0)
 			(effects
@@
 			)
 		)
-		(property "Sheetfile" "pinout2.kicad_sch"
+		(property "Sheetfile" "FPGA_2.kicad_sch"
 			(at 100.33 107.2646 0)
 			(effects
@@
 			(color 0 0 0 0.0000)
 		)
-		(property "Sheetname" "pinout"
+		(property "Sheetname" "FPGA_1"
 			(at 100.33 61.5184 0)
 			(effects
@@
 			)
 		)
-		(property "Sheetfile" "pinout.kicad_sch"
+		(property "Sheetfile" "FPGA_1.kicad_sch"
 			(at 100.33 80.5946 0)
 			(effects
