File: Artix_SOM/Artix_SOM/power.kicad_sch (KiCad schematic)
At the start: 1 part, among them U1 XC7A100T-FGG676

Commit message: update
Parts:
- added C10, C13, C14, C17, C18, C21, C22, C4, C5, C9: 22uF, symbol Device:C
- added C11, C15, C19, C23, C24, C25, C26, C27, C28, C29, C3, C30, C31, C32, C7: 10uF, symbol Device:C
- added C12, C16, C20, C34, C35, C36, C37, C6, C8: 100nF, symbol Device:C
- added D2: LED, symbol Device:LED
- added L1: 2.2uH, symbol Device:L
- added L2, L3, L4, L5: 4.7uH, symbol Device:L
- added R10: 10k., symbol Device:R_US
- added R11, R13, R14, R16, R17, R19, R20, R22, R8: 10k, symbol Device:R_US
- added R12: 13.7k, symbol Device:R_US
- added R15: 33k, symbol Device:R_US
- added R18: 7.5k, symbol Device:R_US
- added R21: 5.76k, symbol Device:R_US
- added R26: 1k, symbol Device:R_US
- added R9: 3.09k, symbol Device:R_US
- added TP1, TP2, TP3, TP4, TP5: TestPoint, symbol Connector:TestPoint
- added U3, U4, U5, U6, U7: TPS563200, Package_TO_SOT_SMD:SOT-23-6, symbol Regulator_Switching:TPS563200
Connections:
- net +1V0: now also C4.1, C5.1, L1.2, R9.1, TP1.1
- net +1V8: now also C10.1, C9.1, L2.2, R12.1, TP2.1
- net GND: now also C10.2, C11.2, C13.2, C14.2, C15.2, C17.2, C18.2, C19.2, C21.2, C22.2, C23.2, C24.2, C25.2, C26.2, C27.2, C28.2, C29.2, C3.2, C30.2, C31.2, C32.2, C34.2, C35.2, C36.2, C37.2, C4.2, C5.2, C7.2, C9.2, D2.1 (K), R10.2, R13.2, R16.2, R19.2, R22.2, U3.1 (GND), U4.1 (GND), U5.1 (GND), U6.1 (GND), U7.1 (GND)
- new net: R8.1, U3.5 (EN)
- new net: R10.1, R9.2, U3.4 (VFB)
- new net: D2.2 (A), R26.2
- new net: R21.2, R22.1, U7.4 (VFB)
- new net: C20.2, L5.1, U7.2 (SW)
- new net: R20.1, U7.5 (EN)
- new net: C20.1, U7.6 (VBST)
- new net: C6.2, L1.1, U3.2 (SW)
- new net: C6.1, U3.6 (VBST)
- new net: R11.1, U4.5 (EN)
- new net: C12.2, L3.1, U5.2 (SW)
- new net: R15.2, R16.1, U5.4 (VFB)
- new net: R14.1, U5.5 (EN)
- new net: C12.1, U5.6 (VBST)
- new net: R18.2, R19.1, U6.4 (VFB)
- new net: R12.2, R13.1, U4.4 (VFB)
- new net: C16.2, L4.1, U6.2 (SW)
- new net: C8.2, L2.1, U4.2 (SW)
- new net: C8.1, U4.6 (VBST)
- new net: C16.1, U6.6 (VBST)
- new net: R17.1, U6.5 (EN)
- new net +1V2: C21.1, C22.1, L5.2, R21.1, TP5.1
- new net +1V35: C17.1, C18.1, L4.2, R18.1, TP4.1
- new net +3V3: C13.1, C14.1, C34.1, C35.1, C36.1, C37.1, L3.2, R15.1, R26.1, TP3.1
- new net +5V: C11.1, C15.1, C19.1, C23.1, C24.1, C25.1, C26.1, C27.1, C28.1, C29.1, C3.1, C30.1, C31.1, C32.1, C7.1, R11.2, R14.2, R17.2, R20.2, R8.2, U3.3 (VIN), U4.3 (VIN), U5.3 (VIN), U6.3 (VIN), U7.3 (VIN)
Other:
- note added: "Vout = 0,768 * (1+ R1/R2)"
- moved on the sheet: U1H

Commit message: update
Changed lines of the file:
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@@
 	)
 	(rectangle
+		(start 163.83 125.73)
+		(end 293.37 170.18)
+		(stroke
+			(width 0)
+			(type dash)
+		)
+		(fill
+			(type none)
+		)
+	)
+	(rectangle
+		(start 163.83 217.17)
+		(end 293.37 269.24)
+		(stroke
+			(width 0)
+			(type dash)
+		)
+		(fill
+			(type none)
+		)
+	)
+	(rectangle
+		(start 163.83 74.93)
+		(end 293.37 124.46)
+		(stroke
+			(width 0)
+			(type dash)
+		)
+		(fill
+			(type none)
+		)
+	)
+	(rectangle
+		(start 163.83 171.45)
+		(end 293.37 215.9)
+		(stroke
+			(width 0)
+			(type dash)
+		)
+		(fill
+			(type none)
+		)
+	)
+	(rectangle
+		(start 163.83 20.32)
+		(end 293.37 72.39)
+		(stroke
+			(width 0)
+			(type dash)
+		)
+		(fill
+			(type none)
+		)
+	)
+	(rectangle
 		(start 160.02 17.78)
 		(end 297.18 279.4)
@@
 		(on_board yes)
 		(dnp no)
-		(fields_autoplaced yes)
 		(property "Reference" "#PWR0113"
 			(at 262.89 172.72 0)
@@
 		)
 		(property "Value" "GND"
-			(at 262.89 171.45 0)
+			(at 258.572 167.132 0)
 			(effects
 				(font
@@
 		(on_board yes)
 		(dnp no)
-		(fields_autoplaced yes)
 		(property "Reference" "C16"
-			(at 245.11 167.64 90)
+			(at 240.538 173.99 90)
 			(effects
 				(font
@@
 		)
 		(property "Value" "100nF"
-			(at 245.11 170.18 90)
+			(at 249.936 174.244 90)
 			(effects
 				(font
@@
 		(on_board yes)
 		(dnp no)
-		(fields_autoplaced yes)
 		(property "Reference" "#PWR0100"
 			(at 262.89 72.39 0)
@@
 		)
 		(property "Value" "GND"
-			(at 262.89 71.12 0)
+			(at 259.08 66.802 0)
 			(effects
 				(font
@@
 		(on_board yes)
 		(dnp no)
-		(fields_autoplaced yes)
 		(property "Reference" "#PWR0125"
 			(at 262.89 270.51 0)
@@
 		)
 		(property "Value" "GND"
-			(at 262.89 269.24 0)
+			(at 258.572 265.684 0)
 			(effects
 				(font
@@
 		(on_board yes)
 		(dnp no)
-		(fields_autoplaced yes)
 		(property "Reference" "#PWR0119"
 			(at 262.89 218.44 0)
@@
 		)
 		(property "Value" "GND"
-			(at 262.89 217.17 0)
+			(at 258.318 213.614 0)
 			(effects
 				(font
@@
 		(on_board yes)
 		(dnp no)
-		(fields_autoplaced yes)
 		(property "Reference" "#PWR099"
 			(at 276.86 68.58 0)
@@
 		)
 		(property "Value" "GND"
-			(at 276.86 67.31 0)
+			(at 280.162 64.262 0)
 			(effects
 				(font
@@
 		(on_board yes)
 		(dnp no)
-		(fields_autoplaced yes)
 		(property "Reference" "C12"
-			(at 245.11 121.92 90)
+			(at 240.284 127.508 90)
 			(effects
 				(font
@@
 		)
 		(property "Value" "100nF"
-			(at 245.11 124.46 90)
+			(at 251.968 127.508 90)
 			(effects
 				(font
@@
 		(on_board yes)
 		(dnp no)
-		(fields_autoplaced yes)
 		(property "Reference" "#PWR0107"
 			(at 262.89 127 0)
@@
 		)
 		(property "Value" "GND"
-			(at 262.89 125.73 0)
+			(at 258.572 120.904 0)
 			(effects
 				(font
