File: Artix_SOM_test/Artix_SOM_test/Artix_SOM_test.kicad_sch (KiCad schematic)
At the start: 0 parts

Commit message: update
Other:
- sheet Test_B1 renamed Test_B1_B2
- sheet Test_B3 renamed Test_B3_B4
- removed sheet Test_B2
- removed sheet Test_B4
- sheet Test_B1_B2: file Test_B1.kicad_sch -> Test_B1_B2.kicad_sch
- sheet Test_B3_B4: file Test_B3.kicad_sch -> Test_B3_B4.kicad_sch
Changed lines of the file:
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@@
 			(color 0 0 0 0.0000)
 		)
-		(property "Sheetname" "Test_B1"
+		(property "Sheetname" "Test_B1_B2"
 			(at 35.56 90.7284 0)
 			(effects
@@
 			)
 		)
-		(property "Sheetfile" "Test_B1.kicad_sch"
+		(property "Sheetfile" "Test_B1_B2.kicad_sch"
 			(at 35.56 107.2646 0)
 			(effects
@@
 				(path "/850c0667-07a1-4e76-ae5f-fa993a9f1707"
 					(page "4")
-				)
-			)
-		)
-	)
-	(sheet
-		(at 68.58 119.38)
-		(size 25.4 15.24)
-		(fields_autoplaced yes)
-		(stroke
-			(width 0.1524)
-			(type solid)
-		)
-		(fill
-			(color 0 0 0 0.0000)
-		)
-		(property "Sheetname" "Test_B4"
-			(at 68.58 118.6684 0)
-			(effects
-				(font
-					(size 1.27 1.27)
-				)
-				(justify left bottom)
-			)
-		)
-		(property "Sheetfile" "Test_B4.kicad_sch"
-			(at 68.58 135.2046 0)
-			(effects
-				(font
-					(size 1.27 1.27)
-				)
-				(justify left top)
-			)
-		)
-		(instances
-			(project "Artix_SOM_test"
-				(path "/850c0667-07a1-4e76-ae5f-fa993a9f1707"
-					(page "7")
 				)
 			)
@@
 	)
 	(sheet
-		(at 35.56 119.38)
+		(at 67.31 91.44)
 		(size 25.4 15.24)
 		(fields_autoplaced yes)
@@
 			(color 0 0 0 0.0000)
 		)
-		(property "Sheetname" "Test_B3"
-			(at 35.56 118.6684 0)
+		(property "Sheetname" "Test_B3_B4"
+			(at 67.31 90.7284 0)
 			(effects
 				(font
@@
 			)
 		)
-		(property "Sheetfile" "Test_B3.kicad_sch"
-			(at 35.56 135.2046 0)
+		(property "Sheetfile" "Test_B3_B4.kicad_sch"
+			(at 67.31 107.2646 0)
 			(effects
 				(font
@@
 				)
 			)
-		)
-	)
-	(sheet
-		(at 68.58 91.44)
-		(size 25.4 15.24)
-		(fields_autoplaced yes)
-		(stroke
-			(width 0.1524)
-			(type solid)
-		)
-		(fill
-			(color 0 0 0 0.0000)
-		)
-		(property "Sheetname" "Test_B2"
-			(at 68.58 90.7284 0)
-			(effects
-				(font
-					(size 1.27 1.27)
-				)
-				(justify left bottom)
-			)
-		)
-		(property "Sheetfile" "Test_B2.kicad_sch"
-			(at 68.58 107.2646 0)
-			(effects
-				(font
-					(size 1.27 1.27)
-				)
-				(justify left top)
-			)
-		)
-		(instances
-			(project "Artix_SOM_test"
-				(path "/850c0667-07a1-4e76-ae5f-fa993a9f1707"
-					(page "5")
-				)
-			)

Commit message: update
Other:
- added sheet External_connections (External_connections.kicad_sch)
Changed lines of the file:
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@@
+	)
+	(sheet
+		(at 100.33 63.5)
+		(size 25.4 15.24)
+		(fields_autoplaced yes)
+		(stroke
+			(width 0.1524)
+			(type solid)
+		)
+		(fill
+			(color 0 0 0 0.0000)
+		)
+		(property "Sheetname" "External_connections"
+			(at 100.33 62.7884 0)
+			(effects
+				(font
+					(size 1.27 1.27)
+				)
+				(justify left bottom)
+			)
+		)
+		(property "Sheetfile" "External_connections.kicad_sch"
+			(at 100.33 79.3246 0)
+			(effects
+				(font
+					(size 1.27 1.27)
+				)
+				(justify left top)
+			)
+		)
+		(instances
+			(project "Artix_SOM_test"
+				(path "/850c0667-07a1-4e76-ae5f-fa993a9f1707"
+					(page "6")
+				)
+			)
+		)
 	)
 	(sheet
@@
 			(project "Artix_SOM_test"
 				(path "/850c0667-07a1-4e76-ae5f-fa993a9f1707"
-					(page "6")
+					(page "5")
 				)
 			)
