File: Artix_SOM_test/Artix_SOM_test/Connector.kicad_sch (KiCad schematic)
At the start: 1 part

Commit message: update
Connections:
- net +5V renamed +12V
Changed lines of the file:
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@@
 	)
 	(global_label "TMS"
-		(shape output)
+		(shape input)
 		(at 109.22 207.01 180)
 		(effects
@@
 	)
 	(symbol
-		(lib_id "power:+5V")
+		(lib_id "power:+12V")
 		(at 133.35 41.91 0)
 		(unit 1)
@@
 		(dnp no)
 		(fields_autoplaced yes)
-		(property "Reference" "#PWR01"
+		(property "Reference" "#PWR05"
 			(at 133.35 45.72 0)
 			(effects
@@
 			)
 		)
-		(property "Value" "+5V"
+		(property "Value" "+12V"
 			(at 133.35 36.83 0)
 			(effects
@@
 			)
 		)
-		(property "Description" "Power symbol creates a global label with name \"+5V\""
+		(property "Description" "Power symbol creates a global label with name \"+12V\""
 			(at 133.35 41.91 0)
 			(effects
@@
 		)
 		(instances
-			(project "Artix_SOM_test"
+			(project ""
 				(path "/850c0667-07a1-4e76-ae5f-fa993a9f1707/8d5f8730-6ad4-4b53-a9a8-f09b304b689f"
-					(reference "#PWR01")
+					(reference "#PWR05")
 					(unit 1)
 				)
