File: Artix_SOM_test/Artix_SOM_test/Connector2.kicad_sch (KiCad schematic)
At the start: 1 part

Commit message: update
Connections:
- net PIN109_B4 is gone; now on net GND: J1.109 (PIN109_B4)
- net PIN110_B4 is gone; now on net GND: J1.110 (PIN110_B4)
- net PIN13_B4 is gone; now on net GND: J1.13 (PIN13_B4)
- net PIN14_B4 is gone; now on net GND: J1.14 (PIN14_B4)
- net PIN1_B4 is gone; now on net GND: J1.1 (PIN1_B4)
- net PIN25_B4 is gone; now on net GND: J1.25 (PIN25_B4)
- net PIN26_B4 is gone; now on net GND: J1.26 (PIN26_B4)
- net PIN2_B4 is gone; now on net GND: J1.2 (PIN2_B4)
- net PIN37_B4 is gone; now on net GND: J1.37 (PIN37_B4)
- net PIN38_B4 is gone; now on net GND: J1.38 (PIN38_B4)
- net PIN49_B4 is gone; now on net GND: J1.49 (PIN49_B4)
- net PIN50_B4 is gone; now on net GND: J1.50 (PIN50_B4)
- net PIN61_B4 is gone; now on net GND: J1.61 (PIN61_B4)
- net PIN62_B4 is gone; now on net GND: J1.62 (PIN62_B4)
- net PIN73_B4 is gone; now on net GND: J1.73 (PIN73_B4)
- net PIN74_B4 is gone; now on net GND: J1.74 (PIN74_B4)
- net PIN85_B4 is gone; now on net GND: J1.85 (PIN85_B4)
- net PIN86_B4 is gone; now on net GND: J1.86 (PIN86_B4)
- net PIN97_B4 is gone; now on net GND: J1.97 (PIN97_B4)
- net PIN98_B4 is gone; now on net GND: J1.98 (PIN98_B4)
- net GND: no longer J1.100 (GND), J1.107 (GND), J1.108 (GND), J1.11 (GND), J1.111 (GND), J1.112 (GND), J1.119 (GND), J1.12 (GND), J1.120 (GND), J1.15 (GND), J1.16 (GND), J1.23 (GND), J1.24 (GND), J1.27 (GND), J1.28 (GND), J1.3 (GND), J1.35 (GND), J1.36 (GND), J1.39 (GND), J1.4 (GND), J1.40 (GND), J1.47 (GND), J1.48 (GND), J1.51 (GND), J1.52 (GND), J1.59 (GND), J1.60 (GND), J1.63 (GND), J1.64 (GND), J1.71 (GND), J1.72 (GND), J1.75 (GND), J1.76 (GND), J1.83 (GND), J1.84 (GND), J1.87 (GND), J1.88 (GND), J1.95 (GND), J1.96 (GND), J1.99 (GND)
- net PIN101_B4: no longer names the net of J1.101 (PIN101_B4)
- net PIN101_B4: now also J1.107 (GND)
- net PIN102_B4: no longer names the net of J1.102 (PIN102_B4)
- net PIN102_B4: now also J1.108 (GND)
- net PIN105_B4: no longer names the net of J1.105 (PIN105_B4)
- net PIN105_B4: now also J1.99 (GND)
- net PIN106_B4: no longer names the net of J1.106 (PIN106_B4)
- net PIN106_B4: now also J1.100 (GND)
- net PIN10_B4: no longer names the net of J1.10 (PIN10_B4)
- net PIN10_B4: now also J1.4 (GND)
- net PIN113_B4 renamed MGTREFCLK0N_3_B4
- net PIN114_B4 renamed MGTREFCLK0N_4_B4
- net PIN117_B4 renamed MGTREFCLK1P_3_B4
- net PIN118_B4 renamed MGTREFCLK1P_4_B4
- net PIN17_B4: no longer names the net of J1.17 (PIN17_B4)
- net PIN17_B4: now also J1.23 (GND)
- net PIN18_B4: no longer names the net of J1.18 (PIN18_B4)
- net PIN18_B4: now also J1.24 (GND)
- net PIN21_B4: no longer names the net of J1.21 (PIN21_B4)
- net PIN21_B4: now also J1.15 (GND)
- net PIN22_B4: no longer names the net of J1.22 (PIN22_B4)
- net PIN22_B4: now also J1.16 (GND)
- net PIN29_B4: no longer names the net of J1.29 (PIN29_B4)
- net PIN29_B4: now also J1.35 (GND)
- net PIN30_B4: no longer names the net of J1.30 (PIN30_B4)
- net PIN30_B4: now also J1.36 (GND)
- net PIN33_B4: no longer names the net of J1.33 (PIN33_B4)
- net PIN33_B4: now also J1.27 (GND)
- net PIN34_B4: no longer names the net of J1.34 (PIN34_B4)
- net PIN34_B4: now also J1.28 (GND)
- net PIN41_B4: no longer names the net of J1.41 (PIN41_B4)
- net PIN41_B4: now also J1.47 (GND)
- net PIN42_B4: no longer names the net of J1.42 (PIN42_B4)
- net PIN42_B4: now also J1.48 (GND)
- net PIN45_B4: no longer names the net of J1.45 (PIN45_B4)
- net PIN45_B4: now also J1.39 (GND)
- net PIN46_B4: no longer names the net of J1.46 (PIN46_B4)
- net PIN46_B4: now also J1.40 (GND)
- net PIN53_B4 renamed MGTREFCLK0N_1_B4
- net PIN54_B4 renamed MGTREFCLK0N_2_B4
- net PIN57_B4 renamed MGTREFCLK1P_1_B4
- net PIN58_B4 renamed MGTREFCLK1P_2_B4
- net PIN5_B4: no longer names the net of J1.5 (PIN5_B4)
- net PIN5_B4: now also J1.11 (GND)
- net PIN65_B4: no longer names the net of J1.65 (PIN65_B4)
- net PIN65_B4: now also J1.71 (GND)
- net PIN66_B4: no longer names the net of J1.66 (PIN66_B4)
- net PIN66_B4: now also J1.72 (GND)
- net PIN69_B4: no longer names the net of J1.69 (PIN69_B4)
- net PIN69_B4: now also J1.63 (GND)
- net PIN6_B4: no longer names the net of J1.6 (PIN6_B4)
- net PIN6_B4: now also J1.12 (GND)
- net PIN70_B4: no longer names the net of J1.70 (PIN70_B4)
- net PIN70_B4: now also J1.64 (GND)
- net PIN77_B4: no longer names the net of J1.77 (PIN77_B4)
- net PIN77_B4: now also J1.83 (GND)
- net PIN78_B4: no longer names the net of J1.78 (PIN78_B4)
- net PIN78_B4: now also J1.84 (GND)
- net PIN81_B4: no longer names the net of J1.81 (PIN81_B4)
- net PIN81_B4: now also J1.75 (GND)
- net PIN82_B4: no longer names the net of J1.82 (PIN82_B4)
- net PIN82_B4: now also J1.76 (GND)
- net PIN89_B4: no longer names the net of J1.89 (PIN89_B4)
- net PIN89_B4: now also J1.95 (GND)
- net PIN90_B4: no longer names the net of J1.90 (PIN90_B4)
- net PIN90_B4: now also J1.96 (GND)
- net PIN93_B4: no longer names the net of J1.93 (PIN93_B4)
- net PIN93_B4: now also J1.87 (GND)
- net PIN94_B4: no longer names the net of J1.94 (PIN94_B4)
- net PIN94_B4: now also J1.88 (GND)
- net PIN9_B4: no longer names the net of J1.9 (PIN9_B4)
- net PIN9_B4: now also J1.3 (GND)
- new net MGTREFCLK0P_1_B4: J1.51 (GND)
- new net MGTREFCLK0P_2_B4: J1.52 (GND)
- new net MGTREFCLK0P_3_B4: J1.111 (GND)
- new net MGTREFCLK0P_4_B4: J1.112 (GND)
- new net MGTREFCLK1N_1_B4: J1.59 (GND)
- new net MGTREFCLK1N_2_B4: J1.60 (GND)
- new net MGTREFCLK1N_3_B4: J1.119 (GND)
- new net MGTREFCLK1N_4_B4: J1.120 (GND)
Other:
- note added: "CLOCK MGT 1 & 2"
- note added: "CLOCK MGT 3 & 4"
